Commit message: Constraint Field RL-Rviz

File: linorobot2_description/urdf/2wd_properties.urdf.xacro (robot description, xacro)
@@ -12,6 +12,6 @@
   <xacro:property name="wheel_mass" value="0.7181" />
   <xacro:property name="wheel_torque" value="0.43" />
-  <xacro:property name="front_caster_wheel" value="false" />
-  <xacro:property name="rear_caster_wheel" value="false" />
+  <xacro:property name="front_caster_wheel" value="true" />
+  <xacro:property name="rear_caster_wheel" value="true" />
   <xacro:property name="wheel_coast" value="-0.0263800000000001" />
   <xacro:property name="laser_pose">

File: linorobot2_description/urdf/mech/base.urdf.xacro (robot description, xacro)
@@ -16,6 +16,7 @@
       </visual>
       <collision>
-        <!-- <origin xyz="-0.0276 0 ${height/2}" rpy="0 0 0"/> -->
-        <origin xyz="0 0 ${height/2-wheel_pos_z}" rpy="0 0 0"/>
+        <!-- base_link is one wheel radius above the footprint. Keep the
+             chassis bottom at base_link z=0 so only the wheels touch ground. -->
+        <origin xyz="0 0 ${height/2}" rpy="0 0 0"/>
         <geometry>
           <box size="${length} ${width} ${height}"/>

File: linorobot2_description/urdf/mech/caster_wheel.urdf.xacro (robot description, xacro)
@@ -6,7 +6,4 @@
       <xacro:property name="caster_wheel_radius" value="0.0325" />
       <xacro:property name="caster_wheel_x" value="-0.0773955999155658" /> <!-- banh sau -->
-      <xacro:property name="caster_wheel_mass" value="1.7181" />
-      <xacro:property name="caster_mesh_file" value="front_caster_wheel.STL" />
-      <xacro:property name="caster_wheel_z" value="-0.026800000000001" />
     </xacro:if>
     <!-- REAR WHEEL CONFIG -->
@@ -14,13 +11,9 @@
       <xacro:property name="caster_wheel_radius" value="0.0325" />
       <xacro:property name="caster_wheel_x" value="0.0639497590100105" />
-      <xacro:property name="caster_wheel_mass" value="1.7191" />
-      <xacro:property name="caster_mesh_file" value="rear_caster_wheel.STL" />
-      <xacro:property name="caster_wheel_z" value="-0.026803000000001" />
     </xacro:if>
     <link name="${side}_caster_wheel_link">
       <visual>
-        <origin xyz="0 0 ${caster_wheel_z}" rpy="0 0 0"/>  <!-- ✅ Để ở (0,0,0) -->
         <geometry>
-            <mesh filename="file://$(find linorobot2_description)/meshes/${caster_mesh_file}" scale="1 1 1"/>
+          <sphere radius="${caster_wheel_radius}"/>
         </geometry>
         <material name="white">
@@ -36,8 +29,8 @@
       <inertial>
         <origin xyz="0 0 0" rpy="0 0 0"/>
-        <mass value="${caster_wheel_mass}"/>
-        <inertia ixx="${(2/5) * caster_wheel_mass * (caster_wheel_radius * caster_wheel_radius)}" ixy="0" ixz="0"
-                 iyy="${(2/5) * caster_wheel_mass * (caster_wheel_radius * caster_wheel_radius)}" iyz="0"
-                 izz="${(2/5) * caster_wheel_mass * (caster_wheel_radius * caster_wheel_radius)}" />
+        <mass value="${mass}"/>
+        <inertia ixx="${(2/5) * mass * (caster_wheel_radius * caster_wheel_radius)}" ixy="0" ixz="0"
+                 iyy="${(2/5) * mass * (caster_wheel_radius * caster_wheel_radius)}" iyz="0"
+                 izz="${(2/5) * mass * (caster_wheel_radius * caster_wheel_radius)}" />
       </inertial>
     </link>
